File: pcb/Washing-Machine-Sensor.kicad_pcb (KiCad board)
At the start: 2 copper layers, 51.8 x 29.8 mm, 23 parts, among them J1 Screw_Terminal_01x02, J2 Conn_02x02_Odd_Even, U1 ESP-12, U2 RFM95W-868S2, U3 AMS1117-3.3, U4 CD4051B

Commit message: Completed Readme, added iBOM
Parts:
- renumbered G*** to G1, G*** to G2
Changed lines of the file:
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@@
     (at 154.7 98.4)
     (attr through_hole)
-    (fp_text reference "G***" (at 0 0) (layer "F.SilkS") hide
+    (fp_text reference "G1" (at 0 0) (layer "F.SilkS") hide
       (effects (font (size 1.524 1.524) (thickness 0.3)))
     )
@@
     (at 162.5 102.1 180)
     (attr board_only exclude_from_pos_files exclude_from_bom)
-    (fp_text reference "G***" (at 1.8 -5.1) (layer "B.Fab")
+    (fp_text reference "G2" (at 1.8 -5.1) (layer "B.Fab")
       (effects (font (size 1.524 1.524) (thickness 0.3)) (justify mirror))
     )
